File: DoubleROM-DOC/DoubleROM-DOC.sch (KiCad schematic (older format))
At the start: 17 parts, among them J1 Bus_ISA_8bit, SW1 ROM 1 Config, SW2 ROM 2 Config, SW4 Size, U1 ROM 1, U2 ROM 2, U3 74LS688, U4 74LS688, U5 74LS33

Commit message: Sunc up PDF and .sch schematic file.
Other:
- note added: "DOC Socket 1"
- note removed: "ROM Socket 1"
Changed lines of the file:
@@
 IBM XT Slot-8 Support
 Text Notes 5300 650  2    50   ~ 0
-ROM Socket 1
+DOC Socket 1
 Text Notes 5300 3700 2    50   ~ 0
 ROM Socket 2
